File: CD4021B-Buttons-Duo.kicad_pcb (KiCad board)
At the start: 2 copper layers, 100 x 50 mm, 50 parts, among them J1 2.54, J10 JST XH, J11 JST XH, J12 JST XH, J13 JST XH, J14 JST XH, J15 JST XH, J16 JST XH, J17 JST XH, J18 3.5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

Commit message: Add voltage divider to the PMOS gate on the board
Parts:
- added D1: Zener, Diodes_SMD:D_SOD-323, B.Cu at (159.5, 121.0)
- added D2: Zener, Diodes_SMD:D_SOD-323, B.Cu at (144.8, 87.8)
- added D3: Zener, Diodes_SMD:D_SOD-323, B.Cu at (148.3, 121.0)
- added D4: Zener, Diodes_SMD:D_SOD-323, B.Cu at (133.6, 87.5)
- added D5: Zener, Diodes_SMD:D_SOD-323, B.Cu at (137.2, 121.0)
- added D6: Zener, Diodes_SMD:D_SOD-323, B.Cu at (122.4, 87.5)
- added D7: Zener, Diodes_SMD:D_SOD-323, B.Cu at (126.0, 121.0)
- added D8: Zener, Diodes_SMD:D_SOD-323, B.Cu at (115.9, 90.9)
- added R10: 0, Resistors_SMD:R_0603_HandSoldering, B.Cu at (146.8, 87.8)
- added R11: 0, Resistors_SMD:R_0603_HandSoldering, B.Cu at (146.3, 121.0)
- added R12: 0, Resistors_SMD:R_0603_HandSoldering, B.Cu at (135.6, 87.5)
- added R13: 0, Resistors_SMD:R_0603_HandSoldering, B.Cu at (135.1, 121.0)
- added R14: 0, Resistors_SMD:R_0603_HandSoldering, B.Cu at (124.5, 87.5)
- added R15: 0, Resistors_SMD:R_0603_HandSoldering, B.Cu at (124.0, 121.0)
- added R16: 0, Resistors_SMD:R_0603_HandSoldering, B.Cu at (113.3, 89.7)
- added R9: 0, Resistors_SMD:R_0603_HandSoldering, B.Cu at (157.5, 121.0)
Connections:
- Q1 pad 3: /LD0 -> Net-(D1-Pad1)
- Q2 pad 3: /LD4 -> Net-(D2-Pad1)
- Q3 pad 3: /LD1 -> Net-(D3-Pad1)
- Q4 pad 3: /LD5 -> Net-(D4-Pad1)
- Q5 pad 3: /LD2 -> Net-(D5-Pad1)
- Q6 pad 3: /LD6 -> Net-(D6-Pad1)
- Q7 pad 3: /LD3 -> Net-(D7-Pad1)
- Q8 pad 3: /LD7 -> Net-(D8-Pad1)
- R1 pad 1: /LD0 -> Net-(D1-Pad1)
- R2 pad 1: /LD4 -> Net-(D2-Pad1)
- R3 pad 1: /LD1 -> Net-(D3-Pad1)
- R4 pad 1: /LD5 -> Net-(D4-Pad1)
- R5 pad 1: /LD2 -> Net-(D5-Pad1)
- R6 pad 1: /LD6 -> Net-(D6-Pad1)
- R7 pad 1: /LD3 -> Net-(D7-Pad1)
- R8 pad 1: /LD7 -> Net-(D8-Pad1)
Routing:
- net Net-(D6-Pad1): track 0.00 -> 6.77 mm
- net Net-(D2-Pad1): track 0.00 -> 6.77 mm
- net Net-(D5-Pad1): track 0.00 -> 6.77 mm
- net Net-(D3-Pad1): track 0.00 -> 6.77 mm
- net Net-(D1-Pad1): track 0.00 -> 6.77 mm
- net Net-(D7-Pad1): track 0.00 -> 6.77 mm
- net Net-(D4-Pad1): track 0.00 -> 6.77 mm
- net Net-(D8-Pad1): track 0.00 -> 5.72 mm
- net /LD7: track 34.3 -> 29.3 mm
- net /LD6: track 22.5 -> 21.5 mm
- net /LD5: track 17.9 -> 16.9 mm
- net /LD4: track 25.2 -> 24.4 mm
- net /LD1: track 17.9 -> 17.2 mm
- net /LD3: track 24.0 -> 23.4 mm
- net /LD0: track 28.1 -> 27.5 mm
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
Commit message: The anode of the zener should be connected to the DRAIN* pin instead of GND
Otherwise the MOSFET always conducts
Parts:
- moved D8 4.64 mm to (111.4, 89.7), turned to 270 degrees
Connections:
- D1 pad 2: GND -> /LD0
- D2 pad 2: GND -> /LD4
- D3 pad 2: GND -> /LD1
- D4 pad 2: GND -> /LD5
- D5 pad 2: GND -> /LD2
- D6 pad 2: GND -> /LD6
- D7 pad 2: GND -> /LD3
- D8 pad 2: GND -> /LD7
Routing:
- net /LD4: track 24.4 -> 26.4 mm
- net /LD1: track 17.2 -> 19.3 mm
- net /LD2: track 19.6 -> 21.6 mm
- net /LD6: track 21.5 -> 23.6 mm
- net /LD0: track 27.5 -> 29.6 mm
- net /LD3: track 23.4 -> 25.4 mm
- net /LD5: track 16.9 -> 19.0 mm
- net /LD7: track 29.3 -> 31.2 mm
Changed lines of the file:
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@@
     (thickness 1.6)
     (drawings 28)
-    (tracks 437)
+    (tracks 453)
     (zones 0)
     (modules 66)
@@
     (pad_to_mask_clearance 0)
     (aux_axis_origin 0 0)
-    (grid_origin 135.636 88.646)
+    (grid_origin 113.284 88.646)
     (visible_elements FFFFFF7F)
     (pcbplotparams
@@
       (net 48 "Net-(D1-Pad1)"))
     (pad 2 smd rect (at 1.05 0 90) (size 0.6 0.45) (layers B.Cu B.Paste B.Mask)
-      (net 2 GND))
+      (net 33 /LD0))
     (model ${KISYS3DMOD}/Diodes_SMD.3dshapes/D_SOD-323.wrl
       (at (xyz 0 0 0))
@@
       (net 49 "Net-(D2-Pad1)"))
     (pad 2 smd rect (at 1.05 0 270) (size 0.6 0.45) (layers B.Cu B.Paste B.Mask)
-      (net 2 GND))
+      (net 34 /LD4))
     (model ${KISYS3DMOD}/Diodes_SMD.3dshapes/D_SOD-323.wrl
       (at (xyz 0 0 0))
@@
       (net 50 "Net-(D3-Pad1)"))
     (pad 2 smd rect (at 1.05 0 90) (size 0.6 0.45) (layers B.Cu B.Paste B.Mask)
-      (net 2 GND))
+      (net 35 /LD1))
     (model ${KISYS3DMOD}/Diodes_SMD.3dshapes/D_SOD-323.wrl
       (at (xyz 0 0 0))
@@
       (net 51 "Net-(D4-Pad1)"))
     (pad 2 smd rect (at 1.05 0 270) (size 0.6 0.45) (layers B.Cu B.Paste B.Mask)
-      (net 2 GND))
+      (net 36 /LD5))
     (model ${KISYS3DMOD}/Diodes_SMD.3dshapes/D_SOD-323.wrl
       (at (xyz 0 0 0))
@@
       (net 52 "Net-(D5-Pad1)"))
     (pad 2 smd rect (at 1.05 0 90) (size 0.6 0.45) (layers B.Cu B.Paste B.Mask)
-      (net 2 GND))
+      (net 37 /LD2))
     (model ${KISYS3DMOD}/Diodes_SMD.3dshapes/D_SOD-323.wrl
       (at (xyz 0 0 0))
@@
       (net 53 "Net-(D6-Pad1)"))
     (pad 2 smd rect (at 1.05 0 270) (size 0.6 0.45) (layers B.Cu B.Paste B.Mask)
-      (net 2 GND))
+      (net 38 /LD6))
     (model ${KISYS3DMOD}/Diodes_SMD.3dshapes/D_SOD-323.wrl
       (at (xyz 0 0 0))
@@
       (net 54 "Net-(D7-Pad1)"))
     (pad 2 smd rect (at 1.05 0 90) (size 0.6 0.45) (layers B.Cu B.Paste B.Mask)
-      (net 2 GND))
+      (net 39 /LD3))
     (model ${KISYS3DMOD}/Diodes_SMD.3dshapes/D_SOD-323.wrl
       (at (xyz 0 0 0))
@@
   )
   (module Diodes_SMD:D_SOD-323 (layer B.Cu)
-    (at 115.858 90.932)
+    (at 111.384 89.696 270)
     (descr SOD-323)
     (tags SOD-323)
     (attr smd)
-    (fp_text reference D8 (at 0 1.85) (layer B.SilkS)
+    (fp_text reference D8 (at 0 1.85 270) (layer B.SilkS)
       (effects (font (size 1 1) (thickness 0.15)) (justify mirror))
     )
-    (fp_text value Zener (at 0.1 -1.9) (layer B.Fab)
+    (fp_text value Zener (at 0.1 -1.9 270) (layer B.Fab)
       (effects (font (size 1 1) (thickness 0.15)) (justify mirror))
     )
-    (fp_text user %R (at 0 1.85) (layer B.Fab)
+    (fp_text user %R (at 0 1.85 270) (layer B.Fab)
       (effects (font (size 1 1) (thickness 0.15)) (justify mirror))
     )
@@
     (fp_line (start -1.5 -0.85) (end 1.05 -0.85) (layer B.SilkS) (width 0.12))
     (fp_line (start -1.5 0.85) (end 1.05 0.85) (layer B.SilkS) (width 0.12))
-    (pad 1 smd rect (at -1.05 0) (size 0.6 0.45) (layers B.Cu B.Paste B.Mask)
+    (pad 1 smd rect (at -1.05 0 270) (size 0.6 0.45) (layers B.Cu B.Paste B.Mask)
       (net 55 "Net-(D8-Pad1)"))
-    (pad 2 smd rect (at 1.05 0) (size 0.6 0.45) (layers B.Cu B.Paste B.Mask)
-      (net 2 GND))
+    (pad 2 smd rect (at 1.05 0 270) (size 0.6 0.45) (layers B.Cu B.Paste B.Mask)
+      (net 40 /LD7))
     (model ${KISYS3DMOD}/Diodes_SMD.3dshapes/D_SOD-323.wrl
       (at (xyz 0 0 0))
@@
   (segment (start 182.88 107.704) (end 188.968 113.792) (width 0.25) (layer F.Cu) (net 32) (status 10))
   (segment (start 188.968 113.792) (end 191.516 113.792) (width 0.25) (layer F.Cu) (net 32) (status 20))
+  (segment (start 159.512 119.988) (end 157.58 119.988) (width 0.25) (layer B.Cu) (net 33))
+  (segment (start 157.58 119.988) (end 157.48 119.888) (width 0.25) (layer B.Cu) (net 33))
   (segment (start 157.48 119.888) (end 157.48 119.038) (width 0.25) (layer B.Cu) (net 33) (status 10))
   (segment (start 157.48 119.038) (end 157.06 118.618) (width 0.25) (layer B.Cu) (net 33))
@@
   (via (at 155.956 118.618) (size 0.6) (drill 0.4) (layers F.Cu B.Cu) (net 33))
   (via (at 151.638 108.458) (size 0.6) (drill 0.4) (layers F.Cu B.Cu) (net 33))
+  (segment (start 144.78 88.8) (end 146.712 88.8) (width 0.25) (layer B.Cu) (net 34))
+  (segment (start 146.712 88.8) (end 146.812 88.9) (width 0.25) (layer B.Cu) (net 34))
   (segment (start 146.812 89.662) (end 146.812 88.9) (width 0.25) (layer B.Cu) (net 34) (status 20))
   (segment (start 147.574 90.424) (end 146.812 89.662) (width 0.25) (layer B.Cu) (net 34))
@@
   (via (at 136.906 98.043992) (size 0.6) (drill 0.4) (layers F.Cu B.Cu) (net 34))
   (via (at 148.336 90.424) (size 0.6) (drill 0.4) (layers F.Cu B.Cu) (net 34))
+  (segment (start 148.336 119.988) (end 146.404 119.988) (width 0.25) (layer B.Cu) (net 35))
+  (segment (start 146.404 119.988) (end 146.304 119.888) (width 0.25) (layer B.Cu) (net 35))
   (segment (start 144.78 118.618) (end 145.796 118.618) (width 0.25) (layer B.Cu) (net 35))
   (segment (start 145.796 118.618) (end 146.304 119.126) (width 0.25) (layer B.Cu) (net 35))
@@
   (segment (start 144.78 118.618) (end 144.769999 118.607999) (width 0.25) (layer F.Cu) (net 35))
   (via (at 144.78 118.618) (size 0.6) (drill 0.4) (layers F.Cu B.Cu) (net 35))
+  (segment (start 133.604 88.546) (end 135.536 88.546) (width 0.25) (layer B.Cu) (net 36))
+  (segment (start 135.536 88.546) (end 135.636 88.646) (width 0.25) (layer B.Cu) (net 36))
   (segment (start 135.636 89.408) (end 135.636 88.646) (width 0.25) (layer B.Cu) (net 36) (status 20))
   (segment (start 136.652 90.424) (end 135.636 89.408) (width 0.25) (layer B.Cu) (net 36))
@@
   (segment (start 137.16 90.424) (end 137.16 95.504) (width 0.25) (layer F.Cu) (net 36))
   (via (at 137.16 90.424) (size 0.6) (drill 0.4) (layers F.Cu B.Cu) (net 36))
+  (segment (start 137.16 119.988) (end 135.228 119.988) (width 0.25) (layer B.Cu) (net 37))
+  (segment (start 135.228 119.988) (end 135.128 119.888) (width 0.25) (layer B.Cu) (net 37))
   (segment (start 133.604 118.618004) (end 134.708004 118.618004) (width 0.25) (layer B.Cu) (net 37))
   (segment (start 134.708004 118.618004) (end 135.128 119.038) (width 0.25) (layer B.Cu) (net 37))
@@
   (via (at 131.064 110.744) (size 0.6) (drill 0.4) (layers F.Cu B.Cu) (net 37))
   (via (at 133.604 118.618004) (size 0.6) (drill 0.4) (layers F.Cu B.Cu) (net 37))
+  (segment (start 122.428 88.546) (end 124.36 88.546) (width 0.25) (layer B.Cu) (net 38))
+  (segment (start 124.36 88.546) (end 124.46 88.646) (width 0.25) (layer B.Cu) (net 38))
   (segment (start 124.46 89.408) (end 124.46 88.646) (width 0.25) (layer B.Cu) (net 38) (status 20))
   (segment (start 125.476 90.424) (end 124.46 89.408) (width 0.25) (layer B.Cu) (net 38))
@@
   (segment (start 127.760002 90.424) (end 131.064 93.727998) (width 0.25) (layer F.Cu) (net 38))
   (via (at 125.984 90.424) (size 0.6) (drill 0.4) (layers F.Cu B.Cu) (net 38))
+  (segment (start 125.984 119.988) (end 124.052 119.988) (width 0.25) (layer B.Cu) (net 39))
+  (segment (start 124.052 119.988) (end 123.952 119.888) (width 0.25) (layer B.Cu) (net 39))
   (segment (start 123.952 119.888) (end 123.952 119.038) (width 0.25) (layer B.Cu) (net 39) (status 10))
   (segment (start 123.952 119.038) (end 123.532 118.618) (width 0.25) (layer B.Cu) (net 39))
@@
   (via (at 126.746 110.744) (size 0.6) (drill 0.4) (layers F.Cu B.Cu) (net 39))
   (via (at 122.428 118.618) (size 0.6) (drill 0.4) (layers F.Cu B.Cu) (net 39))
+  (segment (start 111.384 90.746) (end 113.184 90.746) (width 0.25) (layer B.Cu) (net 40))
+  (segment (start 113.184 90.746) (end 113.284 90.846) (width 0.25) (layer B.Cu) (net 40))
   (segment (start 113.284 92.202) (end 113.284 90.846) (width 0.25) (layer B.Cu) (net 40) (status 20))
   (segment (start 119.887996 98.805996) (end 113.284 92.202) (width 0.25) (layer F.Cu) (net 40))
@@
   (segment (start 125.984 122.088) (end 123.952 122.088) (width 0.25) (layer B.Cu) (net 54) (status 30))
   (segment (start 122.428 119.888) (end 120.518 119.888) (width 0.25) (layer B.Cu) (net 54) (status 30))
-  (segment (start 114.808 88.646) (end 114.808 90.932) (width 0.25) (layer B.Cu) (net 55) (status 30))
+  (segment (start 113.284 88.646) (end 111.384 88.646) (width 0.25) (layer B.Cu) (net 55))
   (segment (start 113.284 88.646) (end 114.808 88.646) (width 0.25) (layer B.Cu) (net 55) (status 30))
   (segment (start 116.718 88.646) (end 114.808 88.646) (width 0.25) (layer B.Cu) (net 55) (status 30))

Commit message: Cleanup: Make LD7 completely on the back side
Routing:
- net /LD7: track 31.2 -> 34.2 mm, vias 2 -> 0
Changed lines of the file:
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@@
     (links 179)
     (no_connects 0)
-    (area 105.334999 78.918999 205.485001 129.069001)
+    (area 97.329048 78.918999 213.490953 129.069001)
     (thickness 1.6)
     (drawings 28)
-    (tracks 453)
+    (tracks 452)
     (zones 0)
     (modules 66)
@@
     (pad_to_mask_clearance 0)
     (aux_axis_origin 0 0)
-    (grid_origin 113.284 88.646)
+    (grid_origin 105.41 78.994)
     (visible_elements FFFFFF7F)
     (pcbplotparams
@@
   (segment (start 182.88 107.704) (end 188.968 113.792) (width 0.25) (layer F.Cu) (net 32) (status 10))
   (segment (start 188.968 113.792) (end 191.516 113.792) (width 0.25) (layer F.Cu) (net 32) (status 20))
-  (segment (start 159.512 119.988) (end 157.58 119.988) (width 0.25) (layer B.Cu) (net 33))
-  (segment (start 157.58 119.988) (end 157.48 119.888) (width 0.25) (layer B.Cu) (net 33))
+  (segment (start 159.512 119.988) (end 157.58 119.988) (width 0.25) (layer B.Cu) (net 33) (status 30))
+  (segment (start 157.58 119.988) (end 157.48 119.888) (width 0.25) (layer B.Cu) (net 33) (status 30))
   (segment (start 157.48 119.888) (end 157.48 119.038) (width 0.25) (layer B.Cu) (net 33) (status 10))
   (segment (start 157.48 119.038) (end 157.06 118.618) (width 0.25) (layer B.Cu) (net 33))
@@
   (via (at 155.956 118.618) (size 0.6) (drill 0.4) (layers F.Cu B.Cu) (net 33))
   (via (at 151.638 108.458) (size 0.6) (drill 0.4) (layers F.Cu B.Cu) (net 33))
-  (segment (start 144.78 88.8) (end 146.712 88.8) (width 0.25) (layer B.Cu) (net 34))
-  (segment (start 146.712 88.8) (end 146.812 88.9) (width 0.25) (layer B.Cu) (net 34))
+  (segment (start 144.78 88.8) (end 146.712 88.8) (width 0.25) (layer B.Cu) (net 34) (status 30))
+  (segment (start 146.712 88.8) (end 146.812 88.9) (width 0.25) (layer B.Cu) (net 34) (status 30))
   (segment (start 146.812 89.662) (end 146.812 88.9) (width 0.25) (layer B.Cu) (net 34) (status 20))
   (segment (start 147.574 90.424) (end 146.812 89.662) (width 0.25) (layer B.Cu) (net 34))
@@
   (via (at 136.906 98.043992) (size 0.6) (drill 0.4) (layers F.Cu B.Cu) (net 34))
   (via (at 148.336 90.424) (size 0.6) (drill 0.4) (layers F.Cu B.Cu) (net 34))
-  (segment (start 148.336 119.988) (end 146.404 119.988) (width 0.25) (layer B.Cu) (net 35))
-  (segment (start 146.404 119.988) (end 146.304 119.888) (width 0.25) (layer B.Cu) (net 35))
+  (segment (start 148.336 119.988) (end 146.404 119.988) (width 0.25) (layer B.Cu) (net 35) (status 30))
+  (segment (start 146.404 119.988) (end 146.304 119.888) (width 0.25) (layer B.Cu) (net 35) (status 30))
   (segment (start 144.78 118.618) (end 145.796 118.618) (width 0.25) (layer B.Cu) (net 35))
   (segment (start 145.796 118.618) (end 146.304 119.126) (width 0.25) (layer B.Cu) (net 35))
@@
   (segment (start 144.78 118.618) (end 144.769999 118.607999) (width 0.25) (layer F.Cu) (net 35))
   (via (at 144.78 118.618) (size 0.6) (drill 0.4) (layers F.Cu B.Cu) (net 35))
-  (segment (start 133.604 88.546) (end 135.536 88.546) (width 0.25) (layer B.Cu) (net 36))
-  (segment (start 135.536 88.546) (end 135.636 88.646) (width 0.25) (layer B.Cu) (net 36))
+  (segment (start 133.604 88.546) (end 135.536 88.546) (width 0.25) (layer B.Cu) (net 36) (status 30))
+  (segment (start 135.536 88.546) (end 135.636 88.646) (width 0.25) (layer B.Cu) (net 36) (status 30))
   (segment (start 135.636 89.408) (end 135.636 88.646) (width 0.25) (layer B.Cu) (net 36) (status 20))
   (segment (start 136.652 90.424) (end 135.636 89.408) (width 0.25) (layer B.Cu) (net 36))
@@
   (segment (start 137.16 90.424) (end 137.16 95.504) (width 0.25) (layer F.Cu) (net 36))
   (via (at 137.16 90.424) (size 0.6) (drill 0.4) (layers F.Cu B.Cu) (net 36))
-  (segment (start 137.16 119.988) (end 135.228 119.988) (width 0.25) (layer B.Cu) (net 37))
-  (segment (start 135.228 119.988) (end 135.128 119.888) (width 0.25) (layer B.Cu) (net 37))
+  (segment (start 137.16 119.988) (end 135.228 119.988) (width 0.25) (layer B.Cu) (net 37) (status 30))
+  (segment (start 135.228 119.988) (end 135.128 119.888) (width 0.25) (layer B.Cu) (net 37) (status 30))
   (segment (start 133.604 118.618004) (end 134.708004 118.618004) (width 0.25) (layer B.Cu) (net 37))
   (segment (start 134.708004 118.618004) (end 135.128 119.038) (width 0.25) (layer B.Cu) (net 37))
@@
   (via (at 131.064 110.744) (size 0.6) (drill 0.4) (layers F.Cu B.Cu) (net 37))
   (via (at 133.604 118.618004) (size 0.6) (drill 0.4) (layers F.Cu B.Cu) (net 37))
-  (segment (start 122.428 88.546) (end 124.36 88.546) (width 0.25) (layer B.Cu) (net 38))
-  (segment (start 124.36 88.546) (end 124.46 88.646) (width 0.25) (layer B.Cu) (net 38))
+  (segment (start 122.428 88.546) (end 124.36 88.546) (width 0.25) (layer B.Cu) (net 38) (status 30))
+  (segment (start 124.36 88.546) (end 124.46 88.646) (width 0.25) (layer B.Cu) (net 38) (status 30))
   (segment (start 124.46 89.408) (end 124.46 88.646) (width 0.25) (layer B.Cu) (net 38) (status 20))
   (segment (start 125.476 90.424) (end 124.46 89.408) (width 0.25) (layer B.Cu) (net 38))
@@
   (segment (start 127.760002 90.424) (end 131.064 93.727998) (width 0.25) (layer F.Cu) (net 38))
   (via (at 125.984 90.424) (size 0.6) (drill 0.4) (layers F.Cu B.Cu) (net 38))
-  (segment (start 125.984 119.988) (end 124.052 119.988) (width 0.25) (layer B.Cu) (net 39))
-  (segment (start 124.052 119.988) (end 123.952 119.888) (width 0.25) (layer B.Cu) (net 39))
+  (segment (start 125.984 119.988) (end 124.052 119.988) (width 0.25) (layer B.Cu) (net 39) (status 30))
+  (segment (start 124.052 119.988) (end 123.952 119.888) (width 0.25) (layer B.Cu) (net 39) (status 30))
   (segment (start 123.952 119.888) (end 123.952 119.038) (width 0.25) (layer B.Cu) (net 39) (status 10))
   (segment (start 123.952 119.038) (end 123.532 118.618) (width 0.25) (layer B.Cu) (net 39))
@@
   (via (at 126.746 110.744) (size 0.6) (drill 0.4) (layers F.Cu B.Cu) (net 39))
   (via (at 122.428 118.618) (size 0.6) (drill 0.4) (layers F.Cu B.Cu) (net 39))
-  (segment (start 111.384 90.746) (end 113.184 90.746) (width 0.25) (layer B.Cu) (net 40))
-  (segment (start 113.184 90.746) (end 113.284 90.846) (width 0.25) (layer B.Cu) (net 40))
-  (segment (start 113.284 92.202) (end 113.284 90.846) (width 0.25) (layer B.Cu) (net 40) (status 20))
-  (segment (start 119.887996 98.805996) (end 113.284 92.202) (width 0.25) (layer F.Cu) (net 40))
-  (segment (start 119.887996 100.076) (end 119.887996 98.805996) (width 0.25) (layer F.Cu) (net 40))
-  (via (at 113.284 92.202) (size 0.6) (drill 0.4) (layers F.Cu B.Cu) (net 40))
   (segment (start 135.89 101.854) (end 135.89 100.838) (width 0.25) (layer B.Cu) (net 40) (status 10))
   (segment (start 135.89 100.838) (end 135.128 100.076) (width 0.25) (layer B.Cu) (net 40))
-  (segment (start 135.128 100.076) (end 119.887996 100.076) (width 0.25) (layer B.Cu) (net 40))
-  (via (at 119.887996 100.076) (size 0.6) (drill 0.4) (layers F.Cu B.Cu) (net 40))
+  (segment (start 135.128 100.076) (end 115.824 100.076) (width 0.25) (layer B.Cu) (net 40))
+  (segment (start 115.824 100.076) (end 115.062 99.314) (width 0.25) (layer B.Cu) (net 40))
+  (segment (start 115.062 99.314) (end 115.062 91.694) (width 0.25) (layer B.Cu) (net 40))
+  (segment (start 115.062 91.694) (end 114.214 90.846) (width 0.25) (layer B.Cu) (net 40))
+  (segment (start 114.214 90.846) (end 113.284 90.846) (width 0.25) (layer B.Cu) (net 40) (status 20))
+  (segment (start 111.384 90.746) (end 113.184 90.746) (width 0.25) (layer B.Cu) (net 40) (status 30))
+  (segment (start 113.184 90.746) (end 113.284 90.846) (width 0.25) (layer B.Cu) (net 40) (status 30))
   (segment (start 177.8 105.918) (end 176.022 104.14) (width 0.25) (layer B.Cu) (net 42))
   (segment (start 176.022 104.14) (end 143.419004 104.14) (width 0.25) (layer B.Cu) (net 42))
@@
   (segment (start 125.984 122.088) (end 123.952 122.088) (width 0.25) (layer B.Cu) (net 54) (status 30))
   (segment (start 122.428 119.888) (end 120.518 119.888) (width 0.25) (layer B.Cu) (net 54) (status 30))
-  (segment (start 113.284 88.646) (end 111.384 88.646) (width 0.25) (layer B.Cu) (net 55))
+  (segment (start 113.284 88.646) (end 111.384 88.646) (width 0.25) (layer B.Cu) (net 55) (status 30))
   (segment (start 113.284 88.646) (end 114.808 88.646) (width 0.25) (layer B.Cu) (net 55) (status 30))
   (segment (start 116.718 88.646) (end 114.808 88.646) (width 0.25) (layer B.Cu) (net 55) (status 30))

Commit message: Cosmetic
Routing:
- net VCC: track 85.7 -> 84.4 mm
Changed lines of the file:
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@@
     (thickness 1.6)
     (drawings 28)
-    (tracks 452)
+    (tracks 453)
     (zones 0)
     (modules 66)
@@
   (gr_line (start 205.41 78.994) (end 205.41 128.994) (layer Edge.Cuts) (width 0.15))
   (gr_line (start 105.41 78.994) (end 205.41 78.994) (layer Edge.Cuts) (width 0.15))
+  (segment (start 163.068 86.614) (end 163.068 95.504) (width 1) (layer F.Cu) (net 1))
+  (segment (start 163.068 95.504) (end 164.338 96.774) (width 1) (layer F.Cu) (net 1))
+  (segment (start 164.338 96.774) (end 170.18 96.774) (width 1) (layer F.Cu) (net 1))
+  (segment (start 170.18 96.774) (end 173.736 100.33) (width 1) (layer F.Cu) (net 1))
+  (segment (start 173.736 100.33) (end 173.736 101.854) (width 0.5) (layer F.Cu) (net 1) (status 20))
   (segment (start 131.318 101.854) (end 130.301996 101.854) (width 0.5) (layer F.Cu) (net 1) (status 10))
   (segment (start 114.3 101.346) (end 129.793996 101.346) (width 1) (layer B.Cu) (net 1))
@@
   (segment (start 112.268 99.314) (end 114.3 101.346) (width 1) (layer B.Cu) (net 1) (status 10))
   (via (at 129.793996 101.346) (size 0.9) (drill 0.6) (layers F.Cu B.Cu) (net 1))
-  (segment (start 172.466 101.854) (end 167.386 101.854) (width 1) (layer F.Cu) (net 1))
-  (segment (start 172.466 101.854) (end 173.736 101.854) (width 0.5) (layer F.Cu) (net 1) (status 20))
   (segment (start 145.796 107.2515) (end 154.241498 107.2515) (width 1) (layer B.Cu) (net 1))
   (segment (start 145.796 107.2515) (end 144.272 107.2515) (width 0.5) (layer B.Cu) (net 1) (status 20))
@@
   (via (at 132.334 106.172) (size 0.6) (drill 0.4) (layers F.Cu B.Cu) (net 1))
   (segment (start 173.736 101.854) (end 175.26 101.854) (width 0.5) (layer F.Cu) (net 1) (status 30))
-  (segment (start 167.386 101.854) (end 161.29 95.758) (width 1) (layer F.Cu) (net 1))
-  (segment (start 161.29 95.758) (end 161.29 86.36) (width 1) (layer F.Cu) (net 1))
   (segment (start 131.318 101.854) (end 133.35 101.854) (width 0.5) (layer F.Cu) (net 1) (status 30))
   (segment (start 150.621986 105.664) (end 149.352 105.664) (width 0.25) (layer F.Cu) (net 2))

Commit message: Update to KiCad 5.0
Routing:
- net GND: track 99.4 -> 5.72 mm

Commit message: Change CSI/CSO to CSB (button)/CSL (lamp) to avoid confusion
Other:
- board text added: "VCC CSL MISO CSB GND"
- board text removed: "VCC CSO MISO CSI GND"
Changed lines of the file:
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@@
     (effects (font (size 1 1) (thickness 0.15)))
   )
-  (gr_text "VCC\nCSO\nMISO\nCSI\nGND" (at 127.254 104.394) (layer B.SilkS)
+  (gr_text "VCC\nCSL\nMISO\nCSB\nGND" (at 127.254 104.394) (layer B.SilkS)
     (effects (font (size 1.5 1.5) (thickness 0.3)) (justify left mirror))
   )
